Commit message: Nov 14th

File: jdamr200_description/urdf/jdamr200.urdf (robot description, URDF)
Before this commit: robot jdamr200, 3 links, 2 joints
Links:
- removed link body_link
- removed link wheel1_link
- removed link wheel2_link
- added link base_footprint
- added link base_link, mass 3.0; collision box size=0.5 0.3 0.15; visual box size=0.5 0.3 0.15
- added link caster_link_front, mass 0.03; collision sphere radius=0.03; visual sphere radius=0.03
- added link caster_link_rear, mass 0.03; collision sphere radius=0.03; visual sphere radius=0.03
- added link laser_link, mass 0.05; collision cylinder length=0.05 radius=0.025; visual cylinder length=0.05 radius=0.025
- added link left_wheel_link, mass 0.0625; collision cylinder length=0.05 radius=0.075; visual cylinder length=0.05 radius=0.075
- added link right_wheel_link, mass 0.0625; collision cylinder length=0.05 radius=0.075; visual cylinder length=0.05 radius=0.075
Joints:
- removed joint wheel1_joint
- removed joint wheel2_joint
- added joint base_joint: type fixed, parent base_footprint, child base_link, origin xyz=0 0 0.075 rpy=0 0 0
- added joint caster_front_joint: type fixed, parent base_link, child caster_link_front, origin xyz=0.2 -0.0 -0.005 rpy=0 0 0
- added joint caster_rear_joint: type fixed, parent base_link, child caster_link_rear, origin xyz=-0.2 -0.0 -0.005 rpy=0 0 0
- added joint laser_joint: type fixed, parent base_link, child laser_link, origin xyz=0.3 0 0.15 rpy=0 0 0
- added joint left_wheel_joint: type continuous, parent base_link, child left_wheel_link, origin xyz=0 0.175 -0.008 rpy=0 0 0, axis 0 1 0
- added joint right_wheel_joint: type continuous, parent base_link, child right_wheel_link, origin xyz=0 -0.175 -0.008 rpy=0 0 0, axis 0 1 0
