Commit message: update jdamr200_description/urdf/jdamr200.urdf to fix the so101_mount_joint origin position, and update jdamr200_gazebo/launch/jdamr200_gazebo.launch.py to replace the SO101_CONTROLLERS_YAML_PATH placeholder with the actual path of the so101_controllers.yaml file.

File: jdamr200_description/urdf/jdamr200_front_arm.urdf (robot description, URDF)
Before this commit: robot jdamr200, 15 links, 14 joints
Joints:
- joint so101_mount_joint: origin xyz=0.15 0 0.075 rpy=0 0 0 -> xyz=0 0 0.075 rpy=0 0 0
